File: kicad-rev2/eload-pwr.kicad_pcb (KiCad board)
At the start: 4 copper layers, 119.5 x 168 mm, 168 parts, among them J1 Barrel_Jack_Switch, J2 USB_C_Receptacle_USB2.0, J3 SWD, J4 Conn_01x01, J5 Conn_01x01, J6 Conn_01x01, J7 Conn_01x01, M1 Fan_4pin, Q101 NMOS, Q102 NMOS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

Commit message: set 22R to 0R (fix for adc)
Parts:
- R14: value 22 -> 0
Changed lines of the file:
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@@
 			)
 		)
-		(property "Value" "22"
+		(property "Value" "0"
 			(at 0 1.65 180)
 			(layer "F.Fab")
